File: PCB/CStick/CStick.kicad_sch (KiCad schematic)
At the start: 6 parts, among them J1 Conn_01x04_Male, U1 Stickbox_Assembly

Commit message: applied footprint changes to all pcbs
forgot to change cstick and motherboard to reflect the new hall sensor footprint, fixed now.
Parts:
- H1: footprint Gamecube MB:MountingHole_1.8mm -> (none)
- H2: footprint Gamecube MB:MountingHole_5.2mm -> (none)
- H3, H4: footprint Gamecube MB:MountingHole_2.0mm -> (none)
- U1: footprint Gamecube MB:GCC_Stickbox_Hall_Only -> (none)
Changed lines of the file:
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@@
       (effects (font (size 1.27 1.27)) (justify left))
     )
-    (property "Footprint" "Gamecube MB:MountingHole_2.0mm" (id 2) (at 91.44 138.43 0)
+    (property "Footprint" "" (id 2) (at 91.44 138.43 0)
       (effects (font (size 1.27 1.27)) hide)
     )
@@
       (effects (font (size 1.27 1.27)) (justify left))
     )
-    (property "Footprint" "Gamecube MB:MountingHole_2.0mm" (id 2) (at 91.44 149.86 0)
+    (property "Footprint" "" (id 2) (at 91.44 149.86 0)
       (effects (font (size 1.27 1.27)) hide)
     )
@@
       (effects (font (size 1.27 1.27)) (justify left))
     )
-    (property "Footprint" "Gamecube MB:GCC_Stickbox_Hall_Only" (id 2) (at 129.54 92.71 0)
+    (property "Footprint" "" (id 2) (at 129.54 92.71 0)
       (effects (font (size 1.27 1.27)) hide)
     )
@@
       (effects (font (size 1.27 1.27)) (justify left))
     )
-    (property "Footprint" "Gamecube MB:MountingHole_5.2mm" (id 2) (at 91.44 127 0)
+    (property "Footprint" "" (id 2) (at 91.44 127 0)
       (effects (font (size 1.27 1.27)) hide)
     )
@@
       (effects (font (size 1.27 1.27)) (justify left))
     )
-    (property "Footprint" "Gamecube MB:MountingHole_1.8mm" (id 2) (at 91.44 115.57 0)
+    (property "Footprint" "" (id 2) (at 91.44 115.57 0)
       (effects (font (size 1.27 1.27)) hide)
     )
@@
     )
     (path "/e42a6a7a-8964-45f9-9ec9-6998e392508a"
-      (reference "H1") (unit 1) (value "MountingHole") (footprint "Gamecube MB:MountingHole_1.8mm")
+      (reference "H1") (unit 1) (value "MountingHole") (footprint "PhobGCC_Footprints:MountingHole_1.8mm")
     )
     (path "/c81d9d6d-1d38-4944-acfb-04c9f7e7b5cc"
-      (reference "H2") (unit 1) (value "MountingHole") (footprint "Gamecube MB:MountingHole_5.2mm")
+      (reference "H2") (unit 1) (value "MountingHole") (footprint "PhobGCC_Footprints:MountingHole_5.2mm")
     )
     (path "/3a568413-17bd-4a87-b1ac-928e77fa1b6a"
-      (reference "H3") (unit 1) (value "MountingHole") (footprint "Gamecube MB:MountingHole_2.0mm")
+      (reference "H3") (unit 1) (value "MountingHole") (footprint "PhobGCC_Footprints:MountingHole_2.0mm")
     )
     (path "/40800b4d-424c-4738-8041-4662989d2010"
-      (reference "H4") (unit 1) (value "MountingHole") (footprint "Gamecube MB:MountingHole_2.0mm")
+      (reference "H4") (unit 1) (value "MountingHole") (footprint "PhobGCC_Footprints:MountingHole_2.0mm")
     )
     (path "/61d7b681-5321-4eb3-aa94-2064a3bbd361"
@@
     )
     (path "/8ae1c09a-53cf-4ff3-980c-45e96b7744a8"
-      (reference "U1") (unit 1) (value "Stickbox_Assembly") (footprint "Gamecube MB:GCC_Stickbox_Hall_Only")
+      (reference "U1") (unit 1) (value "Stickbox_Assembly") (footprint "PhobGCC_Footprints:GCC_Stickbox_Hall_Only")
     )
   )
