File: PCB/KiCad/Motherboard/PhobGCC.kicad_sch (KiCad schematic)
At the start: 80 parts, among them J1 Conn_01x06_Female, J2 Conn_01x04_Female, J3 Conn_01x01_Male, J4 Conn_01x04_Male, J5 Rumble, J6 L, J7 R, Q1 Q_NMOS_GSD, Q2 Q_PMOS_GDS, Q3 Q_NMOS_GSD, SW1 A, SW10 Dup, SW11 Dright, SW12 Ddown, SW13 L, SW14 R, SW2 B, SW3 X, SW4 Y, SW5 Start, SW6 L, SW7 R, SW8 Z, SW9 Dleft, U1 Teensy4.0, U2 2x DRV5053CAQLPGM Hall Effect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, U3 GP2S60-MFG, U4 GP2S60-MFG, U5 Stickbox_Assembly

Commit message: 1.2.2 overhaul
Parts:
- removed D1: (no value), symbol PhobGCC_Symbol_Library:D_Schottky_Shorted
- removed H10: MountingHole, PhobGCC_Footprints:MountingHole_1.8mm, symbol Mechanical:MountingHole
- removed H11: MountingHole, PhobGCC_Footprints:MountingHole_5.2mm, symbol Mechanical:MountingHole
- removed H12, H13: MountingHole, PhobGCC_Footprints:MountingHole_2.0mm, symbol Mechanical:MountingHole
- removed H14, H15: MouseBite, PhobGCC_Footprints:breakaway-mousebites-double, symbol Mechanical:MountingHole
- removed H16: MouseBiteLA, PhobGCC_Footprints:breakaway-mousebites-double, symbol Mechanical:MountingHole
- removed H17: MouseBiteRA, PhobGCC_Footprints:breakaway-mousebites-double, symbol Mechanical:MountingHole
- removed J4: Conn_01x04_Male, Connector_PinHeader_2.00mm:PinHeader_1x04_P2.00mm_Vertical, symbol Connector:Conn_01x04_Male
- removed J6: L, PhobGCC_Footprints:Pin_Header_Straight_1x02_Pitch2.54mm, symbol Connector:Conn_01x02_Male
- removed J7: R, PhobGCC_Footprints:Pin_Header_Straight_1x02_Pitch2.54mm, symbol Connector:Conn_01x02_Male
- removed SW13: L, PhobGCC_Footprints:Trigger_Contact, symbol Switch:SW_Push
- removed SW14: R, PhobGCC_Footprints:Trigger_Contact, symbol Switch:SW_Push
- removed U5: Stickbox_Assembly, PhobGCC_Footprints:GCC_Stickbox_Hall_Only, symbol Gamecube MB:Stickbox_Assembly_Hall_Only
- added D1: D_Schottky_Shorted, PhobGCC_Footprints:D_SOD-523_Shorted, symbol Gamecube MB:D_Schottky_Shorted
- J5: value Rumble -> Conn_01x02_Male
- SW8: value Z -> 1825027-5; symbol PhobGCC_Symbol_Library:SW_DIP_x01 -> Switch:SW_DIP_x01
Connections:
- net Data: now also D1.1 (K), D1.2 (A)
- no-connect marks 4 -> 0
Other:
- moved on the sheet: U2
